Commit message: Heavy-duty version

File: ros2_ws/src/my_car_description/urdf/my_car.urdf.xacro (robot description, xacro)
@@ -2,26 +2,12 @@
 <robot xmlns:xacro="http://www.ros.org/wiki/xacro" name="my_bot">
     <xacro:property name="wheel_offset_x" value="0.2"/>
-    <xacro:property name="wheel_offset_y" value="0.25"/> <xacro:property name="wheel_radius" value="0.06"/>
+    <xacro:property name="wheel_offset_y" value="0.25"/>
+    <xacro:property name="wheel_radius" value="0.06"/>
     <xacro:property name="wheel_width" value="0.04"/>
-    <xacro:property name="wheel_drop" value="0.05"/> <xacro:property name="base_width" value="${2 * wheel_offset_y - wheel_width - 0.05}"/>
+    <xacro:property name="wheel_drop" value="0.05"/>
+    <xacro:property name="base_width" value="${2 * wheel_offset_y - wheel_width - 0.05}"/>
     <xacro:property name="base_length" value="${2 * wheel_offset_x + 0.3}"/>
     <xacro:property name="base_thickness" value="0.02"/>
-    <xacro:property name="stack_length" value="0.4"/>
-    <xacro:property name="stack_width" value="0.25"/>
-    <xacro:property name="level_1_height" value="0.12"/>
-    <xacro:property name="level_2_height" value="0.10"/>
-    <xacro:property name="platform_thickness" value="0.01"/>
-    <xacro:property name="ramp_run" value="${(base_length - stack_length) / 2}"/>
-    <xacro:property name="ramp_rise" value="${level_1_height}"/>
-    <xacro:property name="ramp_length" value="${sqrt(ramp_run*ramp_run + ramp_rise*ramp_rise)}"/>
-    <xacro:property name="ramp_angle" value="${atan2(ramp_rise, ramp_run)}"/>
-    <material name="white"><color rgba="1 1 1 0.8" /></material>
-    <material name="orange"><color rgba="1 0.3 0.1 1"/></material>
-    <material name="blue"><color rgba="0.2 0.2 1 1"/></material>
-    <material name="black"><color rgba="0 0 0 1"/></material>
-    <material name="grey"><color rgba="0.5 0.5 0.5 1"/></material>
-    <material name="metal"><color rgba="0.8 0.8 0.8 1"/></material>
-    <material name="red"><color rgba="1 0 0 1"/></material>
-    <material name="purple"><color rgba="1 0 1 1"/></material> <xacro:macro name="box_inertia" params="m l w h">
+    <xacro:macro name="box_inertia" params="m l w h">
         <inertial>
             <origin xyz="0 0 0" rpy="0 0 0"/>
@@ -37,6 +23,5 @@
         </inertial>
     </xacro:macro>
-    <link name="base_link">
-    </link>
+    <link name="base_link"></link>
     <joint name="supreme_base_joint" type="fixed">
         <parent link="base_link"/>
@@ -45,87 +30,13 @@
     </joint>
     <link name="supreme_base">
-        <visual>
-            <geometry><box size="${base_length} ${base_width} ${base_thickness}"/></geometry>
-            <material name="metal"/>
-        </visual>
-        <collision>
-            <geometry><box size="${base_length} ${base_width} ${base_thickness}"/></geometry>
-        </collision>
+        <visual><geometry><box size="${base_length} ${base_width} ${base_thickness}"/></geometry><material name="Cyan"><color rgba="0 1 1 1"/></material></visual>
+        <collision><geometry><box size="${base_length} ${base_width} ${base_thickness}"/></geometry></collision>
         <xacro:box_inertia m="5.0" l="${base_length}" w="${base_width}" h="${base_thickness}"/>
     </link>
-    <joint name="level_1_joint" type="fixed">
-        <parent link="supreme_base"/>
-        <child link="level_1"/>
-        <origin xyz="0 0 ${base_thickness/2 + level_1_height/2}"/>
-    </joint>
-    <link name="level_1">
-        <visual>
-            <geometry><box size="${stack_length} ${stack_width} ${level_1_height}"/></geometry>
-            <material name="white"/>
-        </visual>
-        <collision>
-            <geometry><box size="${stack_length} ${stack_width} ${level_1_height}"/></geometry>
-        </collision>
-        <xacro:box_inertia m="8.0" l="${stack_length}" w="${stack_width}" h="${level_1_height}"/>
-    </link>
-    <joint name="front_ramp_joint" type="fixed">
-        <parent link="supreme_base"/>
-        <child link="front_ramp"/>
-        <origin xyz="${stack_length/2 + ramp_run/2} 0 ${base_thickness/2 + ramp_rise/2}" rpy="0 ${ramp_angle} 0"/>
-    </joint>
-    <link name="front_ramp">
-        <visual><geometry><box size="${ramp_length} ${stack_width} 0.02"/></geometry><material name="metal"/></visual>
-        <collision><geometry><box size="${ramp_length} ${stack_width} 0.02"/></geometry></collision>
-    </link>
-    <joint name="rear_ramp_joint" type="fixed">
-        <parent link="supreme_base"/>
-        <child link="rear_ramp"/>
-        <origin xyz="-${stack_length/2 + ramp_run/2} 0 ${base_thickness/2 + ramp_rise/2}" rpy="0 -${ramp_angle} 0"/>
-    </joint>
-    <link name="rear_ramp">
-        <visual><geometry><box size="${ramp_length} ${stack_width} 0.02"/></geometry><material name="metal"/></visual>
-        <collision><geometry><box size="${ramp_length} ${stack_width} 0.02"/></geometry></collision>
-    </link>
-    <joint name="platform1_joint" type="fixed">
-        <parent link="level_1"/>
-        <child link="platform_1"/>
-        <origin xyz="0 0 ${level_1_height/2 + platform_thickness/2}"/>
-    </joint>
-    <link name="platform_1">
-        <visual><geometry><box size="${stack_length} ${stack_width} ${platform_thickness}"/></geometry><material name="orange"/></visual>
-    </link>
-    <joint name="level_2_joint" type="fixed">
-        <parent link="platform_1"/>
-        <child link="level_2"/>
-        <origin xyz="0 0 ${platform_thickness/2 + level_2_height/2}"/>
-    </joint>
-    <link name="level_2">
-        <visual>
-            <geometry><box size="${stack_length} ${stack_width} ${level_2_height}"/></geometry>
-            <material name="grey"/>
-        </visual>
-        <collision>
-            <geometry><box size="${stack_length} ${stack_width} ${level_2_height}"/></geometry>
-        </collision>
-        <xacro:box_inertia m="2.0" l="${stack_length}" w="${stack_width}" h="${level_2_height}"/>
-    </link>
-    <joint name="roof_joint" type="fixed">
-        <parent link="level_2"/>
-        <child link="roof"/>
-        <origin xyz="0 0 ${level_2_height/2 + platform_thickness/2}"/>
-    </joint>
-    <link name="roof">
-        <visual><geometry><box size="${stack_length} ${stack_width} ${platform_thickness}"/></geometry><material name="orange"/></visual>
-    </link>
-    <xacro:macro name="wheel" params="name x y">
+    <xacro:macro name="rear_wheel" params="name x y">
         <link name="${name}_wheel">
-            <visual>
-                <geometry><cylinder radius="${wheel_radius}" length="${wheel_width}"/></geometry>
-                <material name="black"/>
-            </visual>
-            <collision>
-                <geometry><cylinder radius="${wheel_radius}" length="${wheel_width}"/></geometry>
-            </collision>
-            <xacro:cylinder_inertia m="0.5" r="${wheel_radius}" h="${wheel_width}"/>
+            <visual><geometry><cylinder radius="${wheel_radius}" length="${wheel_width}"/></geometry><material name="black"><color rgba="0 0 0 1"/></material></visual>
+            <collision><geometry><cylinder radius="${wheel_radius}" length="${wheel_width}"/></geometry></collision>
+            <xacro:cylinder_inertia m="1.5" r="${wheel_radius}" h="${wheel_width}"/>
         </link>
         <joint name="${name}_wheel_joint" type="continuous">
@@ -136,61 +47,37 @@
         </joint>
     </xacro:macro>
-    <link name="left_front_wheel">
-        <visual>
-            <geometry><cylinder radius="${wheel_radius}" length="${wheel_width}"/></geometry>
-            <material name="black"/>
-        </visual>
-        <collision>
-            <geometry><sphere radius="${wheel_radius}"/></geometry>
-        </collision>
-        <xacro:cylinder_inertia m="0.5" r="${wheel_radius}" h="${wheel_width}"/>
-    </link>
-    <joint name="left_front_wheel_joint" type="continuous">
+    <xacro:rear_wheel name="left_rear"   x="-${wheel_offset_x}" y="${wheel_offset_y}"/>
+    <xacro:rear_wheel name="right_rear"  x="-${wheel_offset_x}" y="-${wheel_offset_y}"/>
+    <xacro:macro name="front_wheel" params="name x y">
+        <link name="${name}_wheel">
+            <visual><geometry><cylinder radius="${wheel_radius}" length="${wheel_width}"/></geometry><material name="black"/></visual>
+            <collision><geometry><sphere radius="${wheel_radius}"/></geometry></collision>
+            <xacro:cylinder_inertia m="1.5" r="${wheel_radius}" h="${wheel_width}"/>
+        </link>
+        <joint name="${name}_wheel_joint" type="continuous">
+            <parent link="supreme_base"/>
+            <child link="${name}_wheel"/>
+            <origin xyz="${x} ${y} -${wheel_drop}" rpy="-${pi/2} 0 0"/>
+            <axis xyz="0 0 1"/>
+            <dynamics damping="0.1" friction="0.1"/>
+        </joint>
+    </xacro:macro>
+    <xacro:front_wheel name="left_front"  x="${wheel_offset_x}"  y="${wheel_offset_y}"/>
+    <xacro:front_wheel name="right_front" x="${wheel_offset_x}"  y="-${wheel_offset_y}"/>
+    <joint name="lidar_joint" type="fixed">
         <parent link="supreme_base"/>
-        <child link="left_front_wheel"/>
-        <origin xyz="${wheel_offset_x} ${wheel_offset_y} -${wheel_drop}" rpy="-${pi/2} 0 0"/>
-        <axis xyz="0 0 1"/>
-    </joint>
-    <link name="right_front_wheel">
-        <visual>
-            <geometry><cylinder radius="${wheel_radius}" length="${wheel_width}"/></geometry>
-            <material name="black"/>
-        </visual>
-        <collision>
-            <geometry><sphere radius="${wheel_radius}"/></geometry>
-        </collision>
-        <xacro:cylinder_inertia m="0.5" r="${wheel_radius}" h="${wheel_width}"/>
-    </link>
-    <joint name="right_front_wheel_joint" type="continuous">
-        <parent link="supreme_base"/>
-        <child link="right_front_wheel"/>
-        <origin xyz="${wheel_offset_x} -${wheel_offset_y} -${wheel_drop}" rpy="-${pi/2} 0 0"/>
-        <axis xyz="0 0 1"/>
-    </joint>
-    <xacro:wheel name="left_rear"   x="-${wheel_offset_x}" y="${wheel_offset_y}"/>
-    <xacro:wheel name="right_rear"  x="-${wheel_offset_x}" y="-${wheel_offset_y}"/>
-    <joint name="lidar_joint" type="fixed">
-        <parent link="roof"/>
         <child link="laser_frame"/>
-        <origin xyz="0 0 0.03" rpy="0 0 0"/>
+        <origin xyz="0 0 0.12" rpy="0 0 0"/>
     </joint>
     <link name="laser_frame">
-        <visual><geometry><cylinder radius="0.03" length="0.04"/></geometry><material name="blue"/></visual>
-    </link>
-    <joint name="camera_joint" type="fixed">
-        <parent link="roof"/>
-        <child link="camera_link"/>
-        <origin xyz="${stack_length/2 + 0.01} 0 0.02" rpy="0 0 0"/>
-    </joint>
-    <link name="camera_link">
-        <visual><geometry><box size="0.02 0.04 0.02"/></geometry><material name="red"/></visual>
+        <visual><geometry><cylinder radius="0.03" length="0.04"/></geometry><material name="blue"><color rgba="0 0 1 1"/></material></visual>
     </link>
     <joint name="imu_joint" type="fixed">
-        <parent link="level_2"/>
+        <parent link="supreme_base"/>
         <child link="imu_link"/>
-        <origin xyz="0 0 0.06"/> </joint>
+        <origin xyz="0 0 0.05"/>
+    </joint>
     <link name="imu_link">
-        <visual>
-            <geometry><box size="0.06 0.06 0.06"/></geometry> <material name="purple"/> </visual>
+        <visual><geometry><box size="0.05 0.05 0.05"/></geometry><material name="purple"><color rgba="1 0 1 1"/></material></visual>
     </link>
     <gazebo>
@@ -206,8 +93,7 @@
             <publish_odom>true</publish_odom>
             <publish_odom_tf>true</publish_odom_tf>
-            <publish_wheel_tf>true</publish_wheel_tf>
-        </plugin>
+            <publish_wheel_tf>false</publish_wheel_tf> </plugin>
         <plugin name="gazebo_ros_joint_state_publisher" filename="libgazebo_ros_joint_state_publisher.so">
-            <update_rate>20</update_rate>
+            <update_rate>50</update_rate>
             <joint_name>left_front_wheel_joint</joint_name>
             <joint_name>right_front_wheel_joint</joint_name>
@@ -232,25 +118,3 @@
         </sensor>
     </gazebo>
-    <gazebo reference="camera_link">
-        <sensor name="camera" type="camera">
-            <visualize>true</visualize>
-            <update_rate>10.0</update_rate>
-            <camera>
-                <horizontal_fov>1.089</horizontal_fov>
-                <image><format>R8G8B8</format><width>640</width><height>480</height></image>
-                <clip><near>0.05</near><far>8.0</far></clip>
-            </camera>
-            <plugin name="camera_controller" filename="libgazebo_ros_camera.so">
-                <frame_name>camera_link</frame_name>
-            </plugin>
-        </sensor>
-    </gazebo>
-    <gazebo reference="left_front_wheel">
-        <mu1>0.001</mu1>
-        <mu2>0.001</mu2>
-    </gazebo>
-    <gazebo reference="right_front_wheel">
-        <mu1>0.001</mu1>
-        <mu2>0.001</mu2>
-    </gazebo>
 </robot>

Commit message: Shaking Wheel issue resolved

File: ros2_ws/src/my_car_description/urdf/my_car.urdf.xacro (robot description, xacro)
@@ -9,4 +9,21 @@
     <xacro:property name="base_length" value="${2 * wheel_offset_x + 0.3}"/>
     <xacro:property name="base_thickness" value="0.02"/>
+    <xacro:property name="stack_length" value="0.4"/>
+    <xacro:property name="stack_width" value="0.25"/>
+    <xacro:property name="level_1_height" value="0.12"/>
+    <xacro:property name="level_2_height" value="0.10"/>
+    <xacro:property name="platform_thickness" value="0.01"/>
+    <xacro:property name="ramp_run" value="${(base_length - stack_length) / 2}"/>
+    <xacro:property name="ramp_rise" value="${level_1_height}"/>
+    <xacro:property name="ramp_length" value="${sqrt(ramp_run*ramp_run + ramp_rise*ramp_rise)}"/>
+    <xacro:property name="ramp_angle" value="${atan2(ramp_rise, ramp_run)}"/>
+    <material name="white"><color rgba="1 1 1 0.8"/></material>
+    <material name="orange"><color rgba="1 0.3 0.1 1"/></material>
+    <material name="blue"><color rgba="0.2 0.2 1 1"/></material>
+    <material name="black"><color rgba="0 0 0 1"/></material>
+    <material name="grey"><color rgba="0.5 0.5 0.5 1"/></material>
+    <material name="metal"><color rgba="0.8 0.8 0.8 1"/></material>
+    <material name="red"><color rgba="1 0 0 1"/></material>
+    <material name="purple"><color rgba="1 0 1 1"/></material>
     <xacro:macro name="box_inertia" params="m l w h">
         <inertial>
@@ -30,13 +47,67 @@
     </joint>
     <link name="supreme_base">
-        <visual><geometry><box size="${base_length} ${base_width} ${base_thickness}"/></geometry><material name="Cyan"><color rgba="0 1 1 1"/></material></visual>
+        <visual><geometry><box size="${base_length} ${base_width} ${base_thickness}"/></geometry><material name="metal"/></visual>
         <collision><geometry><box size="${base_length} ${base_width} ${base_thickness}"/></geometry></collision>
         <xacro:box_inertia m="5.0" l="${base_length}" w="${base_width}" h="${base_thickness}"/>
     </link>
+    <joint name="level_1_joint" type="fixed">
+        <parent link="supreme_base"/>
+        <child link="level_1"/>
+        <origin xyz="0 0 ${base_thickness/2 + level_1_height/2}"/>
+    </joint>
+    <link name="level_1">
+        <visual><geometry><box size="${stack_length} ${stack_width} ${level_1_height}"/></geometry><material name="white"/></visual>
+        <collision><geometry><box size="${stack_length} ${stack_width} ${level_1_height}"/></geometry></collision>
+        <xacro:box_inertia m="2.0" l="${stack_length}" w="${stack_width}" h="${level_1_height}"/>
+    </link>
+    <joint name="front_ramp_joint" type="fixed">
+        <parent link="supreme_base"/>
+        <child link="front_ramp"/>
+        <origin xyz="${stack_length/2 + ramp_run/2} 0 ${base_thickness/2 + ramp_rise/2}" rpy="0 ${ramp_angle} 0"/>
+    </joint>
+    <link name="front_ramp">
+        <visual><geometry><box size="${ramp_length} ${stack_width} 0.02"/></geometry><material name="metal"/></visual>
+        <collision><geometry><box size="${ramp_length} ${stack_width} 0.02"/></geometry></collision>
+    </link>
+    <joint name="rear_ramp_joint" type="fixed">
+        <parent link="supreme_base"/>
+        <child link="rear_ramp"/>
+        <origin xyz="-${stack_length/2 + ramp_run/2} 0 ${base_thickness/2 + ramp_rise/2}" rpy="0 -${ramp_angle} 0"/>
+    </joint>
+    <link name="rear_ramp">
+        <visual><geometry><box size="${ramp_length} ${stack_width} 0.02"/></geometry><material name="metal"/></visual>
+        <collision><geometry><box size="${ramp_length} ${stack_width} 0.02"/></geometry></collision>
+    </link>
+    <joint name="platform1_joint" type="fixed">
+        <parent link="level_1"/>
+        <child link="platform_1"/>
+        <origin xyz="0 0 ${level_1_height/2 + platform_thickness/2}"/>
+    </joint>
+    <link name="platform_1">
+        <visual><geometry><box size="${stack_length} ${stack_width} ${platform_thickness}"/></geometry><material name="orange"/></visual>
+    </link>
+    <joint name="level_2_joint" type="fixed">
+        <parent link="platform_1"/>
+        <child link="level_2"/>
+        <origin xyz="0 0 ${platform_thickness/2 + level_2_height/2}"/>
+    </joint>
+    <link name="level_2">
+        <visual><geometry><box size="${stack_length} ${stack_width} ${level_2_height}"/></geometry><material name="grey"/></visual>
+        <collision><geometry><box size="${stack_length} ${stack_width} ${level_2_height}"/></geometry></collision>
+        <xacro:box_inertia m="1.0" l="${stack_length}" w="${stack_width}" h="${level_2_height}"/>
+    </link>
+    <joint name="roof_joint" type="fixed">
+        <parent link="level_2"/>
+        <child link="roof"/>
+        <origin xyz="0 0 ${level_2_height/2 + platform_thickness/2}"/>
+    </joint>
+    <link name="roof">
+        <visual><geometry><box size="${stack_length} ${stack_width} ${platform_thickness}"/></geometry><material name="orange"/></visual>
+    </link>
     <xacro:macro name="rear_wheel" params="name x y">
         <link name="${name}_wheel">
-            <visual><geometry><cylinder radius="${wheel_radius}" length="${wheel_width}"/></geometry><material name="black"><color rgba="0 0 0 1"/></material></visual>
+            <visual><geometry><cylinder radius="${wheel_radius}" length="${wheel_width}"/></geometry><material name="black"/></visual>
             <collision><geometry><cylinder radius="${wheel_radius}" length="${wheel_width}"/></geometry></collision>
-            <xacro:cylinder_inertia m="1.5" r="${wheel_radius}" h="${wheel_width}"/>
+            <xacro:cylinder_inertia m="2.0" r="${wheel_radius}" h="${wheel_width}"/>
         </link>
         <joint name="${name}_wheel_joint" type="continuous">
@@ -45,5 +116,5 @@
             <origin xyz="${x} ${y} -${wheel_drop}" rpy="-${pi/2} 0 0"/>
             <axis xyz="0 0 1"/>
-        </joint>
+            <dynamics damping="0.5" friction="0.2"/> </joint>
     </xacro:macro>
     <xacro:rear_wheel name="left_rear"   x="-${wheel_offset_x}" y="${wheel_offset_y}"/>
@@ -53,5 +124,5 @@
             <visual><geometry><cylinder radius="${wheel_radius}" length="${wheel_width}"/></geometry><material name="black"/></visual>
             <collision><geometry><sphere radius="${wheel_radius}"/></geometry></collision>
-            <xacro:cylinder_inertia m="1.5" r="${wheel_radius}" h="${wheel_width}"/>
+            <xacro:cylinder_inertia m="2.0" r="${wheel_radius}" h="${wheel_width}"/>
         </link>
         <joint name="${name}_wheel_joint" type="continuous">
@@ -60,24 +131,31 @@
             <origin xyz="${x} ${y} -${wheel_drop}" rpy="-${pi/2} 0 0"/>
             <axis xyz="0 0 1"/>
-            <dynamics damping="0.1" friction="0.1"/>
-        </joint>
+            <dynamics damping="0.5" friction="0.2"/> </joint>
     </xacro:macro>
     <xacro:front_wheel name="left_front"  x="${wheel_offset_x}"  y="${wheel_offset_y}"/>
     <xacro:front_wheel name="right_front" x="${wheel_offset_x}"  y="-${wheel_offset_y}"/>
     <joint name="lidar_joint" type="fixed">
-        <parent link="supreme_base"/>
+        <parent link="roof"/>
         <child link="laser_frame"/>
-        <origin xyz="0 0 0.12" rpy="0 0 0"/>
+        <origin xyz="0 0 0.03" rpy="0 0 0"/>
     </joint>
     <link name="laser_frame">
-        <visual><geometry><cylinder radius="0.03" length="0.04"/></geometry><material name="blue"><color rgba="0 0 1 1"/></material></visual>
+        <visual><geometry><cylinder radius="0.03" length="0.04"/></geometry><material name="blue"/></visual>
+    </link>
+    <joint name="camera_joint" type="fixed">
+        <parent link="roof"/>
+        <child link="camera_link"/>
+        <origin xyz="${stack_length/2 + 0.01} 0 0.02" rpy="0 0 0"/>
+    </joint>
+    <link name="camera_link">
+        <visual><geometry><box size="0.02 0.04 0.02"/></geometry><material name="red"/></visual>
     </link>
     <joint name="imu_joint" type="fixed">
-        <parent link="supreme_base"/>
+        <parent link="level_2"/>
         <child link="imu_link"/>
         <origin xyz="0 0 0.05"/>
     </joint>
     <link name="imu_link">
-        <visual><geometry><box size="0.05 0.05 0.05"/></geometry><material name="purple"><color rgba="1 0 1 1"/></material></visual>
+        <visual><geometry><box size="0.05 0.05 0.05"/></geometry><material name="purple"/></visual>
     </link>
     <gazebo>
@@ -93,5 +171,6 @@
             <publish_odom>true</publish_odom>
             <publish_odom_tf>true</publish_odom_tf>
-            <publish_wheel_tf>false</publish_wheel_tf> </plugin>
+            <publish_wheel_tf>false</publish_wheel_tf>
+        </plugin>
         <plugin name="gazebo_ros_joint_state_publisher" filename="libgazebo_ros_joint_state_publisher.so">
             <update_rate>50</update_rate>
@@ -118,3 +197,17 @@
         </sensor>
     </gazebo>
+    <gazebo reference="camera_link">
+        <sensor name="camera" type="camera">
+            <visualize>true</visualize>
+            <update_rate>10.0</update_rate>
+            <camera>
+                <horizontal_fov>1.089</horizontal_fov>
+                <image><format>R8G8B8</format><width>640</width><height>480</height></image>
+                <clip><near>0.05</near><far>8.0</far></clip>
+            </camera>
+            <plugin name="camera_controller" filename="libgazebo_ros_camera.so">
+                <frame_name>camera_link</frame_name>
+            </plugin>
+        </sensor>
+    </gazebo>
 </robot>
