Commit message: Imu Sensor repositioned

File: ros2_ws/src/my_car_description/urdf/my_car.urdf.xacro (robot description, xacro)
@@ -1,4 +1,4 @@
 <?xml version="1.0"?>
-<robot xmlns:xacro="http://www.ros.org/wiki/xacro" name="my_bot">
+<robot xmlns:xacro="http://www.ros.org/wiki/xacro" name="my_car">
     <xacro:property name="wheel_offset_x" value="0.2"/>
     <xacro:property name="wheel_offset_y" value="0.25"/>
@@ -12,5 +12,5 @@
     <xacro:property name="stack_width" value="0.25"/>
     <xacro:property name="level_1_height" value="0.12"/>
-    <xacro:property name="level_2_height" value="0.10"/>
+    <xacro:property name="level_2_height" value="0.12"/>
     <xacro:property name="platform_thickness" value="0.01"/>
     <xacro:property name="ramp_run" value="${(base_length - stack_length) / 2}"/>
@@ -154,5 +154,5 @@
         <parent link="level_2"/>
         <child link="imu_link"/>
-        <origin xyz="0 0 0.05"/>
+        <origin xyz="0 0 -0.034"/>
     </joint>
     <link name="imu_link">

Commit message: Added Transparency to view inner parts

File: ros2_ws/src/my_car_description/urdf/my_car.urdf.xacro (robot description, xacro)
@@ -57,5 +57,5 @@
     </joint>
     <link name="level_1">
-        <visual><geometry><box size="${stack_length} ${stack_width} ${level_1_height}"/></geometry><material name="white"/></visual>
+        <visual><geometry><box size="${stack_length} ${stack_width} ${level_1_height}"/></geometry><material name="metal"/></visual>
         <collision><geometry><box size="${stack_length} ${stack_width} ${level_1_height}"/></geometry></collision>
         <xacro:box_inertia m="2.0" l="${stack_length}" w="${stack_width}" h="${level_1_height}"/>
@@ -93,5 +93,5 @@
     </joint>
     <link name="level_2">
-        <visual><geometry><box size="${stack_length} ${stack_width} ${level_2_height}"/></geometry><material name="grey"/></visual>
+        <visual><geometry><box size="${stack_length} ${stack_width} ${level_2_height}"/></geometry><material name="metal"/></visual>
         <collision><geometry><box size="${stack_length} ${stack_width} ${level_2_height}"/></geometry></collision>
         <xacro:box_inertia m="1.0" l="${stack_length}" w="${stack_width}" h="${level_2_height}"/>

Commit message: Colour Enhanced, torques increased  and Friction Added in Wheels

File: ros2_ws/src/my_car_description/urdf/my_car.urdf.xacro (robot description, xacro)
@@ -165,5 +165,5 @@
             <wheel_separation>${2 * wheel_offset_y}</wheel_separation>
             <wheel_diameter>${2 * wheel_radius}</wheel_diameter>
-            <max_wheel_torque>200</max_wheel_torque>
+            <max_wheel_torque>500</max_wheel_torque>
             <max_wheel_acceleration>10.0</max_wheel_acceleration>
             <odometry_frame>odom</odometry_frame>
@@ -233,3 +233,59 @@
         </sensor>
     </gazebo>
+    <gazebo reference="supreme_base">
+        <material>Gazebo/Grey</material>
+    </gazebo>
+    <gazebo reference="level_1">
+        <material>Gazebo/Grey</material>
+    </gazebo>
+    <gazebo reference="front_ramp">
+        <material>Gazebo/Grey</material>
+    </gazebo>
+    <gazebo reference="rear_ramp">
+        <material>Gazebo/Grey</material>
+    </gazebo>
+    <gazebo reference="level_2">
+        <material>Gazebo/Grey</material>
+    </gazebo>
+    <gazebo reference="platform_1">
+        <material>Gazebo/Orange</material>
+    </gazebo>
+    <gazebo reference="roof">
+        <material>Gazebo/Orange</material>
+    </gazebo>
+    <gazebo reference="left_rear_wheel">
+        <material>Gazebo/FlatBlack</material>
+    </gazebo>
+    <gazebo reference="right_rear_wheel">
+        <material>Gazebo/FlatBlack</material>
+    </gazebo>
+    <gazebo reference="left_front_wheel">
+        <material>Gazebo/FlatBlack</material>
+    </gazebo>
+    <gazebo reference="right_front_wheel">
+        <material>Gazebo/FlatBlack</material>
+    </gazebo>
+    <gazebo reference="laser_frame">
+        <material>Gazebo/Blue</material>
+    </gazebo>
+    <gazebo reference="camera_link">
+        <material>Gazebo/Red</material>
+    </gazebo>
+    <gazebo reference="imu_link">
+        <material>Gazebo/Purple</material>
+    </gazebo>
+    <gazebo reference="left_rear_wheel">
+        <mu1>1.0</mu1> <mu2>1.0</mu2> <kp>1000000.0</kp> <kd>100.0</kd> </gazebo>
+    <gazebo reference="right_rear_wheel">
+        <mu1>1.0</mu1> <mu2>1.0</mu2>
+        <kp>1000000.0</kp> <kd>100.0</kd>
+    </gazebo>
+    <gazebo reference="left_front_wheel">
+        <mu1>1.0</mu1> <mu2>1.0</mu2>
+        <kp>1000000.0</kp> <kd>100.0</kd>
+    </gazebo>
+    <gazebo reference="right_front_wheel">
+        <mu1>1.0</mu1> <mu2>1.0</mu2>
+        <kp>1000000.0</kp> <kd>100.0</kd>
+    </gazebo>
 </robot>
