Commit message: updated URDF with real mechanical dimenstions

File: ros2_ws/src/my_car_description/urdf/my_car.urdf (robot description, URDF)
Before this commit: robot my_car, 15 links, 14 joints
Links:
- link front_ramp: geometry collision box size=0.2 0.2 0.02; visual box size=0.2 0.2 0.02
- link left_front_wheel: mass 2.0 -> 0.5
- link level_1: geometry collision box size=0.3 0.2 0.12; visual box size=0.3 0.2 0.12
- link level_2: geometry collision box size=0.3 0.2 0.12; visual box size=0.3 0.2 0.12
- link platform_1: geometry visual box size=0.3 0.2 0.01
- link rear_ramp: geometry collision box size=0.2 0.2 0.02; visual box size=0.2 0.2 0.02
- link right_front_wheel: mass 2.0 -> 0.5
- link roof: geometry visual box size=0.3 0.2 0.01
- link supreme_base: mass 5.0 -> 2.0; geometry collision box size=0.69 0.25 0.02; visual box size=0.69 0.25 0.02
Joints:
- joint camera_joint: origin xyz=0.21000000000000002 0 0.02 rpy=0 0 0 -> xyz=0.16 0 0.02 rpy=0 0 0
- joint front_ramp_joint: origin xyz=0.275 0 0.06999999999999999 rpy=0 0.6747409422235527 0 -> xyz=0.23 0 0.06999999999999999 rpy=0 0.6435011087932843 0
- joint left_front_wheel_joint: origin xyz=0.2 0.25 -0.05 rpy=-1.5707963267948966 0 0 -> xyz=0.25 0.18 -0.05 rpy=-1.5707963267948966 0 0
- joint left_rear_wheel_joint: origin xyz=-0.2 0.25 -0.05 rpy=-1.5707963267948966 0 0 -> xyz=-0.25 0.18 -0.05 rpy=-1.5707963267948966 0 0
- joint rear_ramp_joint: origin xyz=-0.275 0 0.06999999999999999 rpy=0 -0.6747409422235527 0 -> xyz=-0.23 0 0.06999999999999999 rpy=0 -0.6435011087932843 0
- joint right_front_wheel_joint: origin xyz=0.2 -0.25 -0.05 rpy=-1.5707963267948966 0 0 -> xyz=0.25 -0.18 -0.05 rpy=-1.5707963267948966 0 0
- joint right_rear_wheel_joint: origin xyz=-0.2 -0.25 -0.05 rpy=-1.5707963267948966 0 0 -> xyz=-0.25 -0.18 -0.05 rpy=-1.5707963267948966 0 0

File: ros2_ws/src/my_car_description/urdf/my_car.urdf.xacro (robot description, xacro)
@@ -1,20 +1,20 @@
 <?xml version="1.0"?>
 <robot xmlns:xacro="http://www.ros.org/wiki/xacro" name="my_car">
-    <xacro:property name="wheel_offset_x" value="0.2"/>
-    <xacro:property name="wheel_offset_y" value="0.25"/>
+   <xacro:property name="wheel_offset_y" value="0.18"/>
+    <xacro:property name="wheel_offset_x" value="0.25"/>
     <xacro:property name="wheel_radius" value="0.06"/>
     <xacro:property name="wheel_width" value="0.04"/>
     <xacro:property name="wheel_drop" value="0.05"/>
-    <xacro:property name="base_width" value="${2 * wheel_offset_y - wheel_width - 0.05}"/>
-    <xacro:property name="base_length" value="${2 * wheel_offset_x + 0.3}"/>
+    <xacro:property name="base_width" value="0.25"/>
+    <xacro:property name="base_length" value="0.69"/>
     <xacro:property name="base_thickness" value="0.02"/>
-    <xacro:property name="stack_length" value="0.4"/>
-    <xacro:property name="stack_width" value="0.25"/>
+    <xacro:property name="stack_length" value="0.30"/>
+    <xacro:property name="stack_width" value="0.20"/>
     <xacro:property name="level_1_height" value="0.12"/>
     <xacro:property name="level_2_height" value="0.12"/>
     <xacro:property name="platform_thickness" value="0.01"/>
-    <xacro:property name="ramp_run" value="${(base_length - stack_length) / 2}"/>
+    <xacro:property name="ramp_length" value="0.20"/>
     <xacro:property name="ramp_rise" value="${level_1_height}"/>
-    <xacro:property name="ramp_length" value="${sqrt(ramp_run*ramp_run + ramp_rise*ramp_rise)}"/>
+    <xacro:property name="ramp_run" value="${sqrt(ramp_length*ramp_length - ramp_rise*ramp_rise)}"/>
     <xacro:property name="ramp_angle" value="${atan2(ramp_rise, ramp_run)}"/>
     <material name="white"><color rgba="1 1 1 0.8"/></material>
@@ -49,5 +49,5 @@
         <visual><geometry><box size="${base_length} ${base_width} ${base_thickness}"/></geometry><material name="metal"/></visual>
         <collision><geometry><box size="${base_length} ${base_width} ${base_thickness}"/></geometry></collision>
-        <xacro:box_inertia m="5.0" l="${base_length}" w="${base_width}" h="${base_thickness}"/>
+        <xacro:box_inertia m="2.0" l="${base_length}" w="${base_width}" h="${base_thickness}"/>
     </link>
     <joint name="level_1_joint" type="fixed">
@@ -124,5 +124,5 @@
             <visual><geometry><cylinder radius="${wheel_radius}" length="${wheel_width}"/></geometry><material name="black"/></visual>
             <collision><geometry><sphere radius="${wheel_radius}"/></geometry></collision>
-            <xacro:cylinder_inertia m="2.0" r="${wheel_radius}" h="${wheel_width}"/>
+            <xacro:cylinder_inertia m="0.5" r="${wheel_radius}" h="${wheel_width}"/>
         </link>
         <joint name="${name}_wheel_joint" type="continuous">

Commit message: GNSS added

File: ros2_ws/src/my_car_description/urdf/my_car.urdf (robot description, URDF)
Before this commit: robot my_car, 15 links, 14 joints
Links:
- added link gnss_link; visual cylinder length=0.02 radius=0.02
Joints:
- added joint gnss_joint: type fixed, parent roof, child gnss_link, origin xyz=-0.12 0 0.015 rpy=0 0 0
- joint camera_joint: origin xyz=0.16 0 0.02 rpy=0 0 0 -> xyz=0.16 0 0.015 rpy=0 0 0
- joint lidar_joint: origin xyz=0 0 0.03 rpy=0 0 0 -> xyz=0 0 0.025 rpy=0 0 0

File: ros2_ws/src/my_car_description/urdf/my_car.urdf.xacro (robot description, xacro)
@@ -1,5 +1,5 @@
 <?xml version="1.0"?>
 <robot xmlns:xacro="http://www.ros.org/wiki/xacro" name="my_car">
-   <xacro:property name="wheel_offset_y" value="0.18"/>
+    <xacro:property name="wheel_offset_y" value="0.18"/>
     <xacro:property name="wheel_offset_x" value="0.25"/>
     <xacro:property name="wheel_radius" value="0.06"/>
@@ -26,4 +26,5 @@
     <material name="red"><color rgba="1 0 0 1"/></material>
     <material name="purple"><color rgba="1 0 1 1"/></material>
+    <material name="yellow"><color rgba="1 1 0 1"/></material>
     <xacro:macro name="box_inertia" params="m l w h">
         <inertial>
@@ -116,5 +117,6 @@
             <origin xyz="${x} ${y} -${wheel_drop}" rpy="-${pi/2} 0 0"/>
             <axis xyz="0 0 1"/>
-            <dynamics damping="0.5" friction="0.2"/> </joint>
+            <dynamics damping="0.5" friction="0.2"/>
+        </joint>
     </xacro:macro>
     <xacro:rear_wheel name="left_rear"   x="-${wheel_offset_x}" y="${wheel_offset_y}"/>
@@ -131,5 +133,6 @@
             <origin xyz="${x} ${y} -${wheel_drop}" rpy="-${pi/2} 0 0"/>
             <axis xyz="0 0 1"/>
-            <dynamics damping="0.5" friction="0.2"/> </joint>
+            <dynamics damping="0.5" friction="0.2"/>
+        </joint>
     </xacro:macro>
     <xacro:front_wheel name="left_front"  x="${wheel_offset_x}"  y="${wheel_offset_y}"/>
@@ -138,5 +141,5 @@
         <parent link="roof"/>
         <child link="laser_frame"/>
-        <origin xyz="0 0 0.03" rpy="0 0 0"/>
+        <origin xyz="0 0 0.025" rpy="0 0 0"/>
     </joint>
     <link name="laser_frame">
@@ -146,5 +149,5 @@
         <parent link="roof"/>
         <child link="camera_link"/>
-        <origin xyz="${stack_length/2 + 0.01} 0 0.02" rpy="0 0 0"/>
+        <origin xyz="${stack_length/2 + 0.01} 0 0.015" rpy="0 0 0"/>
     </joint>
     <link name="camera_link">
@@ -158,4 +161,12 @@
     <link name="imu_link">
         <visual><geometry><box size="0.05 0.05 0.05"/></geometry><material name="purple"/></visual>
+    </link>
+    <joint name="gnss_joint" type="fixed">
+        <parent link="roof"/>
+        <child link="gnss_link"/>
+        <origin xyz="-0.12 0 0.015" rpy="0 0 0"/>
+    </joint>
+    <link name="gnss_link">
+        <visual><geometry><cylinder radius="0.02" length="0.02"/></geometry><material name="yellow"/></visual>
     </link>
     <gazebo>
@@ -233,59 +244,43 @@
         </sensor>
     </gazebo>
-    <gazebo reference="supreme_base">
-        <material>Gazebo/Grey</material>
-    </gazebo>
-    <gazebo reference="level_1">
-        <material>Gazebo/Grey</material>
-    </gazebo>
-    <gazebo reference="front_ramp">
-        <material>Gazebo/Grey</material>
-    </gazebo>
-    <gazebo reference="rear_ramp">
-        <material>Gazebo/Grey</material>
-    </gazebo>
-    <gazebo reference="level_2">
-        <material>Gazebo/Grey</material>
-    </gazebo>
-    <gazebo reference="platform_1">
-        <material>Gazebo/Orange</material>
-    </gazebo>
-    <gazebo reference="roof">
-        <material>Gazebo/Orange</material>
-    </gazebo>
+    <gazebo reference="gnss_link">
+        <sensor name="gnss_sensor" type="gps">
+            <always_on>true</always_on>
+            <update_rate>5.0</update_rate>
+            <plugin name="gnss_controller" filename="libgazebo_ros_gps_sensor.so">
+                <ros>
+                    <remapping>~/out:=/gnss/fix</remapping>
+                </ros>
+                <output_type>sensor_msgs/NavSatFix</output_type>
+                <frame_name>gnss_link</frame_name>
+            </plugin>
+        </sensor>
+    </gazebo>
+    <gazebo reference="supreme_base"><material>Gazebo/Grey</material></gazebo>
+    <gazebo reference="front_ramp"><material>Gazebo/Grey</material></gazebo>
+    <gazebo reference="rear_ramp"><material>Gazebo/Grey</material></gazebo>
+    <gazebo reference="level_1"><material>Gazebo/Grey</material></gazebo>
+    <gazebo reference="level_2"><material>Gazebo/Grey</material></gazebo>
+    <gazebo reference="platform_1"><material>Gazebo/Orange</material></gazebo>
+    <gazebo reference="roof"><material>Gazebo/Orange</material></gazebo>
+    <gazebo reference="laser_frame"><material>Gazebo/Blue</material></gazebo>
+    <gazebo reference="camera_link"><material>Gazebo/Red</material></gazebo>
+    <gazebo reference="imu_link"><material>Gazebo/Purple</material></gazebo>
+    <gazebo reference="gnss_link"><material>Gazebo/Yellow</material></gazebo>
     <gazebo reference="left_rear_wheel">
         <material>Gazebo/FlatBlack</material>
+        <mu1>1.0</mu1><mu2>1.0</mu2><kp>1000000.0</kp><kd>100.0</kd>
     </gazebo>
     <gazebo reference="right_rear_wheel">
         <material>Gazebo/FlatBlack</material>
+        <mu1>1.0</mu1><mu2>1.0</mu2><kp>1000000.0</kp><kd>100.0</kd>
     </gazebo>
     <gazebo reference="left_front_wheel">
         <material>Gazebo/FlatBlack</material>
+        <mu1>1.0</mu1><mu2>1.0</mu2><kp>1000000.0</kp><kd>100.0</kd>
     </gazebo>
     <gazebo reference="right_front_wheel">
         <material>Gazebo/FlatBlack</material>
-    </gazebo>
-    <gazebo reference="laser_frame">
-        <material>Gazebo/Blue</material>
-    </gazebo>
-    <gazebo reference="camera_link">
-        <material>Gazebo/Red</material>
-    </gazebo>
-    <gazebo reference="imu_link">
-        <material>Gazebo/Purple</material>
-    </gazebo>
-    <gazebo reference="left_rear_wheel">
-        <mu1>1.0</mu1> <mu2>1.0</mu2> <kp>1000000.0</kp> <kd>100.0</kd> </gazebo>
-    <gazebo reference="right_rear_wheel">
-        <mu1>1.0</mu1> <mu2>1.0</mu2>
-        <kp>1000000.0</kp> <kd>100.0</kd>
-    </gazebo>
-    <gazebo reference="left_front_wheel">
-        <mu1>1.0</mu1> <mu2>1.0</mu2>
-        <kp>1000000.0</kp> <kd>100.0</kd>
-    </gazebo>
-    <gazebo reference="right_front_wheel">
-        <mu1>1.0</mu1> <mu2>1.0</mu2>
-        <kp>1000000.0</kp> <kd>100.0</kd>
+        <mu1>1.0</mu1><mu2>1.0</mu2><kp>1000000.0</kp><kd>100.0</kd>
     </gazebo>
 </robot>

Commit message: Setting up Workspace

File: ros2_ws/src/my_car_description/urdf/my_car.urdf (robot description, URDF)
Before this commit: robot my_car, 16 links, 15 joints
Links:
- link front_ramp: geometry collision box size=0.2 0.2 0.02; visual box size=0.2 0.2 0.02
- link left_front_wheel: mass 2.0 -> 0.5
- link level_1: geometry collision box size=0.3 0.2 0.12; visual box size=0.3 0.2 0.12
- link level_2: geometry collision box size=0.3 0.2 0.12; visual box size=0.3 0.2 0.12
- link platform_1: geometry visual box size=0.3 0.2 0.01
- link rear_ramp: geometry collision box size=0.2 0.2 0.02; visual box size=0.2 0.2 0.02
- link right_front_wheel: mass 2.0 -> 0.5
- link roof: geometry visual box size=0.3 0.2 0.01
- link supreme_base: mass 5.0 -> 2.0; geometry collision box size=0.69 0.25 0.02; visual box size=0.69 0.25 0.02
Joints:
- joint camera_joint: origin xyz=0.21000000000000002 0 0.015 rpy=0 0 0 -> xyz=0.16 0 0.015 rpy=0 0 0
- joint front_ramp_joint: origin xyz=0.275 0 0.06999999999999999 rpy=0 0.6747409422235527 0 -> xyz=0.23 0 0.06999999999999999 rpy=0 0.6435011087932843 0
- joint left_front_wheel_joint: origin xyz=0.2 0.25 -0.05 rpy=-1.5707963267948966 0 0 -> xyz=0.25 0.18 -0.05 rpy=-1.5707963267948966 0 0
- joint left_rear_wheel_joint: origin xyz=-0.2 0.25 -0.05 rpy=-1.5707963267948966 0 0 -> xyz=-0.25 0.18 -0.05 rpy=-1.5707963267948966 0 0
- joint rear_ramp_joint: origin xyz=-0.275 0 0.06999999999999999 rpy=0 -0.6747409422235527 0 -> xyz=-0.23 0 0.06999999999999999 rpy=0 -0.6435011087932843 0
- joint right_front_wheel_joint: origin xyz=0.2 -0.25 -0.05 rpy=-1.5707963267948966 0 0 -> xyz=0.25 -0.18 -0.05 rpy=-1.5707963267948966 0 0
- joint right_rear_wheel_joint: origin xyz=-0.2 -0.25 -0.05 rpy=-1.5707963267948966 0 0 -> xyz=-0.25 -0.18 -0.05 rpy=-1.5707963267948966 0 0

File: ros2_ws/src/my_car_description/urdf/my_car.urdf.xacro (robot description, xacro)
@@ -1,20 +1,20 @@
 <?xml version="1.0"?>
 <robot xmlns:xacro="http://www.ros.org/wiki/xacro" name="my_car">
-    <xacro:property name="wheel_offset_x" value="0.2"/>
-    <xacro:property name="wheel_offset_y" value="0.25"/>
+    <xacro:property name="wheel_offset_y" value="0.18"/>
+    <xacro:property name="wheel_offset_x" value="0.25"/>
     <xacro:property name="wheel_radius" value="0.06"/>
     <xacro:property name="wheel_width" value="0.04"/>
     <xacro:property name="wheel_drop" value="0.05"/>
-    <xacro:property name="base_width" value="${2 * wheel_offset_y - wheel_width - 0.05}"/>
-    <xacro:property name="base_length" value="${2 * wheel_offset_x + 0.3}"/>
+    <xacro:property name="base_width" value="0.25"/>
+    <xacro:property name="base_length" value="0.69"/>
     <xacro:property name="base_thickness" value="0.02"/>
-    <xacro:property name="stack_length" value="0.4"/>
-    <xacro:property name="stack_width" value="0.25"/>
+    <xacro:property name="stack_length" value="0.30"/>
+    <xacro:property name="stack_width" value="0.20"/>
     <xacro:property name="level_1_height" value="0.12"/>
     <xacro:property name="level_2_height" value="0.12"/>
     <xacro:property name="platform_thickness" value="0.01"/>
-    <xacro:property name="ramp_run" value="${(base_length - stack_length) / 2}"/>
+    <xacro:property name="ramp_length" value="0.20"/>
     <xacro:property name="ramp_rise" value="${level_1_height}"/>
-    <xacro:property name="ramp_length" value="${sqrt(ramp_run*ramp_run + ramp_rise*ramp_rise)}"/>
+    <xacro:property name="ramp_run" value="${sqrt(ramp_length*ramp_length - ramp_rise*ramp_rise)}"/>
     <xacro:property name="ramp_angle" value="${atan2(ramp_rise, ramp_run)}"/>
     <material name="white"><color rgba="1 1 1 0.8"/></material>
@@ -50,5 +50,5 @@
         <visual><geometry><box size="${base_length} ${base_width} ${base_thickness}"/></geometry><material name="metal"/></visual>
         <collision><geometry><box size="${base_length} ${base_width} ${base_thickness}"/></geometry></collision>
-        <xacro:box_inertia m="5.0" l="${base_length}" w="${base_width}" h="${base_thickness}"/>
+        <xacro:box_inertia m="2.0" l="${base_length}" w="${base_width}" h="${base_thickness}"/>
     </link>
     <joint name="level_1_joint" type="fixed">
@@ -58,5 +58,5 @@
     </joint>
     <link name="level_1">
-        <visual><geometry><box size="${stack_length} ${stack_width} ${level_1_height}"/></geometry><material name="white"/></visual>
+        <visual><geometry><box size="${stack_length} ${stack_width} ${level_1_height}"/></geometry><material name="metal"/></visual>
         <collision><geometry><box size="${stack_length} ${stack_width} ${level_1_height}"/></geometry></collision>
         <xacro:box_inertia m="2.0" l="${stack_length}" w="${stack_width}" h="${level_1_height}"/>
@@ -94,5 +94,5 @@
     </joint>
     <link name="level_2">
-        <visual><geometry><box size="${stack_length} ${stack_width} ${level_2_height}"/></geometry><material name="grey"/></visual>
+        <visual><geometry><box size="${stack_length} ${stack_width} ${level_2_height}"/></geometry><material name="metal"/></visual>
         <collision><geometry><box size="${stack_length} ${stack_width} ${level_2_height}"/></geometry></collision>
         <xacro:box_inertia m="1.0" l="${stack_length}" w="${stack_width}" h="${level_2_height}"/>
@@ -126,5 +126,5 @@
             <visual><geometry><cylinder radius="${wheel_radius}" length="${wheel_width}"/></geometry><material name="black"/></visual>
             <collision><geometry><sphere radius="${wheel_radius}"/></geometry></collision>
-            <xacro:cylinder_inertia m="2.0" r="${wheel_radius}" h="${wheel_width}"/>
+            <xacro:cylinder_inertia m="0.5" r="${wheel_radius}" h="${wheel_width}"/>
         </link>
         <joint name="${name}_wheel_joint" type="continuous">
@@ -176,5 +176,5 @@
             <wheel_separation>${2 * wheel_offset_y}</wheel_separation>
             <wheel_diameter>${2 * wheel_radius}</wheel_diameter>
-            <max_wheel_torque>200</max_wheel_torque>
+            <max_wheel_torque>500</max_wheel_torque>
             <max_wheel_acceleration>10.0</max_wheel_acceleration>
             <odometry_frame>odom</odometry_frame>
@@ -267,5 +267,6 @@
     <gazebo reference="camera_link"><material>Gazebo/Red</material></gazebo>
     <gazebo reference="imu_link"><material>Gazebo/Purple</material></gazebo>
-    <gazebo reference="gnss_link"><material>Gazebo/Yellow</material></gazebo> <gazebo reference="left_rear_wheel">
+    <gazebo reference="gnss_link"><material>Gazebo/Yellow</material></gazebo>
+    <gazebo reference="left_rear_wheel">
         <material>Gazebo/FlatBlack</material>
         <mu1>1.0</mu1>
